File: ButtonPushing/SolenoidDriver/Solenoids.sch (EAGLE design)
At the start: 29 parts, among them U1 TLE94112EL

Commit message: Fully routed PCB
Basically done, but needs to be checked over
Parts:
- removed C2, C3: 100nF, rcl:C-EUC0402
- removed D12: 1N5819-B, diode:1N5819-B
- added C5, C6: 100nF, rcl:C-EUC0402K
- added CSN, EN, GND, NC, SCLK, SDI, SDO, VCC, VSOLENOID: (no value), wirepad:1,6/0,8
- added D13: MBR0520LT, diode:MBR0520LT
- C1: device rcl:C-EUC0402 -> rcl:C-EUC0402K
- D1, D10, D11, D2, D3, D4, D5, D6, D7, D8, D9: value 1N5819-B -> MBR0520LT; device diode:1N5819-B -> diode:MBR0520LT
Connections:
- removed net CS: U1.CSN
- removed net EN: U1.EN
- removed net MISO: U1.SDO
- removed net MOSI: U1.SDI
- removed net SCK: U1.SCLK
- removed net SOLENOID: C1.1, C2.1, C4.1, U1.VS1, U1.VS2
- new net N$22: EN.P, U1.EN
- new net N$23: CSN.P, U1.CSN
- new net N$24: SCLK.P, U1.SCLK
- new net N$25: SDI.P, U1.SDI
- new net N$26: SDO.P, U1.SDO
- new net VDD: C1.1, C4.1, C5.1, U1.VS1, U1.VS2, VSOLENOID.P
- net GND: now also C5.2, C6.2, D13.A, GND.P, NC.P; no longer C2.2, C3.2, D12.A
- net N$1: now also D13.C; no longer D1.C
- net N$10: now also D9.C; no longer D10.C
- net N$11: now also D10.C; no longer D11.C
- net N$12: now also D11.C; no longer D12.C
- net N$2: now also D1.C; no longer D2.C
- net N$3: now also D2.C; no longer D3.C
- net N$4: now also D3.C; no longer D4.C
- net N$5: now also D4.C; no longer D5.C
- net N$6: now also D5.C; no longer D6.C
- net N$7: now also D6.C; no longer D7.C
- net N$8: now also D7.C; no longer D8.C
- net N$9: now also D8.C; no longer D9.C
- net VCC: now also C6.1, VCC.P; no longer C3.1
Other:
- moved on the sheet: C1, C4

Commit message: Built version revision 1
Parts:
- added D12: MBRA340T3, diode:MBRA340T3
- added GND1, GND2: (no value), wirepad:1,6/0,8
- added H1, H2, H3, H4: MOUNT-HOLE2.8, holes:MOUNT-HOLE2.8
Connections:
- net GND: now also D12.A, GND1.P, GND2.P; no longer NC.P
- net VDD: now also D12.C
Changed lines of the file:
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@@
 <part name="NC" library="wirepad" deviceset="1,6/0,8" device=""/>
 <part name="SUPPLY23" library="supply2" deviceset="GND" device=""/>
+<part name="GND1" library="wirepad" deviceset="1,6/0,8" device=""/>
+<part name="SUPPLY24" library="supply2" deviceset="GND" device=""/>
+<part name="GND2" library="wirepad" deviceset="1,6/0,8" device=""/>
+<part name="SOL4" library="supply1" deviceset="VDD" device="" value="Vsolenoid"/>
+<part name="SUPPLY25" library="supply2" deviceset="GND" device=""/>
+<part name="D12" library="diode" deviceset="MBRA340T3" device=""/>
+<part name="H1" library="holes" deviceset="MOUNT-HOLE" device="2.8"/>
+<part name="H2" library="holes" deviceset="MOUNT-HOLE" device="2.8"/>
+<part name="H3" library="holes" deviceset="MOUNT-HOLE" device="2.8"/>
+<part name="H4" library="holes" deviceset="MOUNT-HOLE" device="2.8"/>
 </parts>
 <sheets>
@@
 <instance part="SOL3" gate="G$1" x="78.74" y="88.9"/>
 <instance part="NC" gate="P" x="48.26" y="91.44" rot="R270"/>
-<instance part="SUPPLY23" gate="GND" x="48.26" y="86.36"/>
+<instance part="SUPPLY23" gate="GND" x="33.02" y="86.36"/>
+<instance part="GND1" gate="P" x="33.02" y="91.44" rot="R270"/>
+<instance part="SUPPLY24" gate="GND" x="27.94" y="86.36"/>
+<instance part="GND2" gate="P" x="27.94" y="91.44" rot="R270"/>
+<instance part="SOL4" gate="G$1" x="55.88" y="104.14"/>
+<instance part="SUPPLY25" gate="GND" x="55.88" y="93.98"/>
+<instance part="D12" gate="G$1" x="55.88" y="99.06" rot="R90"/>
+<instance part="H1" gate="G$1" x="5.08" y="76.2"/>
+<instance part="H2" gate="G$1" x="5.08" y="71.12"/>
+<instance part="H3" gate="G$1" x="5.08" y="66.04"/>
+<instance part="H4" gate="G$1" x="5.08" y="60.96"/>
 </instances>
 <busses>
@@
 <pinref part="SUPPLY6" gate="GND" pin="GND"/>
 <pinref part="SUPPLY7" gate="GND" pin="GND"/>
-<junction x="73.66" y="17.78"/>
 </segment>
 <segment>
@@
 </segment>
 <segment>
-<pinref part="NC" gate="P" pin="P"/>
 <pinref part="SUPPLY23" gate="GND" pin="GND"/>
+<pinref part="GND1" gate="P" pin="P"/>
+</segment>
+<segment>
+<pinref part="SUPPLY24" gate="GND" pin="GND"/>
+<pinref part="GND2" gate="P" pin="P"/>
+</segment>
+<segment>
+<pinref part="SUPPLY25" gate="GND" pin="GND"/>
+<pinref part="D12" gate="G$1" pin="A"/>
 </segment>
 </net>
@@
 <pinref part="C4" gate="G$1" pin="1"/>
 <pinref part="SOL3" gate="G$1" pin="VDD"/>
+</segment>
+<segment>
+<pinref part="SOL4" gate="G$1" pin="VDD"/>
+<pinref part="D12" gate="G$1" pin="C"/>
 </segment>
 </net>
@@
 </sheet>
 </sheets>
+<errors>
+</errors>
 </schematic>
 </drawing>
